File: hardware/recorder/Recorder.brd (EAGLE design)
At the start: 66.5 x 73.7 mm, 23 parts, among them U1 PDM1-S5-D12-S, U2 LM6132BIN, U3 Value, U4 L7908CV, U5 L7808ABV, U6 ZVN4424A, U7 TEENSY_3.6_DIL

Commit message: Update recorder hardware
Parts:
- R3: value 300R -> 330R
- moved R_GAIN 3.69 mm to (49.8, 19.2)
- moved R_SHUNT 0.51 mm to (39.3, 11.6)
- renumbered HARVESTER to HARVESTER_TERMINAL
Routing:
- net N$3: track 8.07 -> 4.35 mm
- net N$1: track 8.12 -> 4.66 mm
Other:
- board text added: "SOCRAETES Recorder V 1.1.4 University of Duisburg-Essen Networked Embedded Systems (NES)"
- board text removed: "SOCRAETES Recorder (Rev 0.3) University of Duisburg-Essen Networked Embedded Systems (NES)"
Changed lines of the file:
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@@
 <plain>
 <text x="62.23" y="29.21" size="1.778" layer="25" rot="R90">HRVST +      -</text>
-<text x="58.4708" y="27.94" size="1.016" layer="25" rot="R270">SOCRAETES Recorder (Rev 0.3)
+<text x="58.4708" y="27.94" size="1.016" layer="25" rot="R270">SOCRAETES Recorder V 1.1.4
 University of Duisburg-Essen
 Networked Embedded Systems (NES)</text>
@@
 <attribute name="POPULARITY" value="6" x="22.86" y="127" size="1.778" layer="27" rot="R180" display="off"/>
 </element>
-<element name="HARVESTER" library="con-ptr500" library_urn="urn:adsk.eagle:library:181" package="AK300/2" package3d_urn="urn:adsk.eagle:package:9881/1" value="" x="53.34" y="41.91" smashed="yes" rot="R90">
+<element name="HARVESTER_TERMINAL" library="con-ptr500" library_urn="urn:adsk.eagle:library:181" package="AK300/2" package3d_urn="urn:adsk.eagle:package:9881/1" value="" x="53.34" y="41.91" smashed="yes" rot="R90">
 <attribute name="MF" value="" x="59.69" y="85.09" size="1.778" layer="27" rot="R90" display="off"/>
 <attribute name="MPN" value="" x="59.69" y="85.09" size="1.778" layer="27" rot="R90" display="off"/>
@@
 <attribute name="VALUE" x="31.115" y="26.6954" size="1.27" layer="27" ratio="10" rot="R90"/>
 </element>
-<element name="R3" library="rcl" library_urn="urn:adsk.eagle:library:334" package="0207/10" package3d_urn="urn:adsk.eagle:package:23491/2" value="300R" x="27.94" y="48.26" smashed="yes" rot="R180">
+<element name="R3" library="rcl" library_urn="urn:adsk.eagle:library:334" package="0207/10" package3d_urn="urn:adsk.eagle:package:23491/2" value="330R" x="27.94" y="48.26" smashed="yes" rot="R180">
 <attribute name="NAME" x="28.956" y="46.736" size="1.27" layer="25" ratio="10" rot="R180"/>
 <attribute name="POPULARITY" value="81" x="-29.21" y="143.51" size="1.778" layer="27" rot="R180" display="off"/>
@@
 <attribute name="VALUE" x="30.2006" y="48.895" size="1.27" layer="27" ratio="10" rot="R180"/>
 </element>
-<element name="R_GAIN" library="rcl" library_urn="urn:adsk.eagle:library:334" package="0207/10" package3d_urn="urn:adsk.eagle:package:23491/2" value="" x="49.53" y="22.86" smashed="yes" rot="R180">
-<attribute name="NAME" x="52.705" y="26.162" size="1.27" layer="25" ratio="10" rot="R180"/>
-<attribute name="POPULARITY" value="81" x="30.48" y="123.19" size="1.778" layer="27" rot="R180" display="off"/>
-<attribute name="SPICEPREFIX" value="R" x="30.48" y="123.19" size="1.778" layer="27" rot="R180" display="off"/>
-<attribute name="VALUE" x="51.7906" y="23.495" size="1.27" layer="27" ratio="10" rot="R180"/>
-</element>
-<element name="R_SHUNT" library="rcl" library_urn="urn:adsk.eagle:library:334" package="0207/10" package3d_urn="urn:adsk.eagle:package:23491/2" value="" x="39.2684" y="12.1412" smashed="yes" rot="R90">
-<attribute name="NAME" x="37.2364" y="8.0772" size="1.27" layer="25" ratio="10" rot="R90"/>
-<attribute name="POPULARITY" value="81" x="134.5184" y="31.1912" size="1.778" layer="27" rot="R90" display="off"/>
-<attribute name="SPICEPREFIX" value="R" x="134.5184" y="31.1912" size="1.778" layer="27" rot="R90" display="off"/>
-<attribute name="VALUE" x="39.9034" y="9.8806" size="1.27" layer="27" ratio="10" rot="R90"/>
+<element name="R_GAIN" library="rcl" library_urn="urn:adsk.eagle:library:334" package="0207/10" package3d_urn="urn:adsk.eagle:package:23491/2" value="" x="49.784" y="19.177" smashed="yes" rot="R180">
+<attribute name="NAME" x="52.959" y="22.479" size="1.27" layer="25" ratio="10" rot="R180"/>
+<attribute name="POPULARITY" value="81" x="30.734" y="119.507" size="1.778" layer="27" rot="R180" display="off"/>
+<attribute name="SPICEPREFIX" value="R" x="30.734" y="119.507" size="1.778" layer="27" rot="R180" display="off"/>
+<attribute name="VALUE" x="52.0446" y="19.812" size="1.27" layer="27" ratio="10" rot="R180"/>
+</element>
+<element name="R_SHUNT" library="rcl" library_urn="urn:adsk.eagle:library:334" package="0207/10" package3d_urn="urn:adsk.eagle:package:23491/2" value="" x="39.2684" y="11.6332" smashed="yes" rot="R90">
+<attribute name="NAME" x="37.2364" y="7.5692" size="1.27" layer="25" ratio="10" rot="R90"/>
+<attribute name="POPULARITY" value="81" x="134.5184" y="30.6832" size="1.778" layer="27" rot="R90" display="off"/>
+<attribute name="SPICEPREFIX" value="R" x="134.5184" y="30.6832" size="1.778" layer="27" rot="R90" display="off"/>
+<attribute name="VALUE" x="39.9034" y="9.3726" size="1.27" layer="27" ratio="10" rot="R90"/>
 </element>
 <element name="U6" library="NES_Solar_Cell_Recorder_And_Emulator" package="TO92-CBE" value="ZVN4424A" x="30.48" y="13.1572" smashed="yes" rot="R270">
@@
 <contactref element="C4" pad="+"/>
 <contactref element="U2" pad="4"/>
-<contactref element="HARVESTER" pad="2"/>
+<contactref element="HARVESTER_TERMINAL" pad="2"/>
 <contactref element="C6" pad="-"/>
 <contactref element="D1" pad="A"/>
@@
 </signal>
 <signal name="HARVESTER+">
-<contactref element="HARVESTER" pad="1"/>
+<contactref element="HARVESTER_TERMINAL" pad="1"/>
 <contactref element="R_SHUNT" pad="1"/>
 <contactref element="U3" pad="3"/>
@@
 <wire x1="42.9" y1="41.63" x2="44.45" y2="43.18" width="0.5" layer="16"/>
 <wire x1="42.9" y1="37.19" x2="42.9" y2="41.63" width="0.5" layer="16"/>
-<wire x1="39.2684" y1="7.0612" x2="40.8432" y2="8.636" width="0.5" layer="1"/>
-<wire x1="44.3484" y1="8.636" x2="46.1264" y2="10.414" width="0.5" layer="1"/>
-<wire x1="40.8432" y1="8.636" x2="44.3484" y2="8.636" width="0.5" layer="1"/>
+<wire x1="39.2684" y1="6.5532" x2="39.3192" y2="6.604" width="0.5" layer="1"/>
+<wire x1="41.148" y1="6.604" x2="44.958" y2="10.414" width="0.5" layer="1"/>
+<wire x1="44.958" y1="10.414" x2="46.1264" y2="10.414" width="0.5" layer="1"/>
+<wire x1="39.3192" y1="6.604" x2="41.148" y2="6.604" width="0.5" layer="1"/>
 </signal>
 <signal name="N$1">
 <contactref element="R_GAIN" pad="2"/>
 <contactref element="U3" pad="1"/>
-<wire x1="44.55" y1="16.84" x2="44.55" y2="22.34" width="0.5" layer="1"/>
-<wire x1="45.65" y1="15.74" x2="44.55" y2="16.84" width="0.5" layer="1"/>
-<wire x1="44.55" y1="22.34" x2="44.45" y2="22.86" width="0.5" layer="1"/>
-<wire x1="45.65" y1="15.74" x2="46.1264" y2="15.494" width="0.5" layer="1"/>
+<wire x1="44.704" y1="19.177" x2="44.704" y2="16.256" width="0.5" layer="1"/>
+<wire x1="44.704" y1="16.256" x2="45.466" y2="15.494" width="0.5" layer="1"/>
+<wire x1="45.466" y1="15.494" x2="46.1264" y2="15.494" width="0.5" layer="1"/>
 </signal>
 <signal name="N$3">
 <contactref element="R_GAIN" pad="1"/>
 <contactref element="U3" pad="8"/>
-<wire x1="54.45" y1="21.24" x2="54.45" y2="22.34" width="0.5" layer="1"/>
-<wire x1="53.35" y1="20.14" x2="54.45" y2="21.24" width="0.5" layer="1"/>
-<wire x1="53.35" y1="15.74" x2="53.35" y2="20.14" width="0.5" layer="1"/>
-<wire x1="54.45" y1="22.34" x2="54.61" y2="22.86" width="0.5" layer="1"/>
-<wire x1="53.35" y1="15.74" x2="53.7464" y2="15.494" width="0.5" layer="1"/>
+<wire x1="54.864" y1="19.177" x2="54.864" y2="16.256" width="0.5" layer="1"/>
+<wire x1="54.864" y1="16.256" x2="54.102" y2="15.494" width="0.5" layer="1"/>
+<wire x1="54.102" y1="15.494" x2="53.7464" y2="15.494" width="0.5" layer="1"/>
 </signal>
 <signal name="N$6">
@@
 <contactref element="R_SHUNT" pad="2"/>
 <contactref element="U3" pad="2"/>
-<wire x1="33" y1="10.79" x2="30.8" y2="10.79" width="0.5" layer="1"/>
-<wire x1="39.05" y1="16.84" x2="33" y2="10.79" width="0.5" layer="1"/>
-<wire x1="30.8" y1="10.79" x2="30.48" y2="10.6172" width="0.5" layer="1"/>
-<wire x1="39.05" y1="16.84" x2="39.2684" y2="17.2212" width="0.5" layer="1"/>
-<wire x1="43.45" y1="12.99" x2="45.65" y2="12.99" width="0.5" layer="1"/>
-<wire x1="39.6" y1="16.84" x2="43.45" y2="12.99" width="0.5" layer="1"/>
-<wire x1="45.65" y1="12.99" x2="46.1264" y2="12.954" width="0.5" layer="1"/>
-<wire x1="39.6" y1="16.84" x2="39.2684" y2="17.2212" width="0.5" layer="1"/>
+<wire x1="39.2684" y1="16.7132" x2="41.1988" y2="16.7132" width="0.5" layer="1"/>
+<wire x1="44.958" y1="12.954" x2="46.1264" y2="12.954" width="0.5" layer="1"/>
+<wire x1="41.1988" y1="16.7132" x2="44.958" y2="12.954" width="0.5" layer="1"/>
+<wire x1="37.592" y1="15.748" x2="37.592" y2="14.224" width="0.5" layer="1"/>
+<wire x1="37.592" y1="15.748" x2="38.5572" y2="16.7132" width="0.5" layer="1"/>
+<wire x1="38.5572" y1="16.7132" x2="39.2684" y2="16.7132" width="0.5" layer="1"/>
+<wire x1="33.9852" y1="10.6172" x2="30.48" y2="10.6172" width="0.5" layer="1"/>
+<wire x1="37.592" y1="14.224" x2="33.9852" y2="10.6172" width="0.5" layer="1"/>
 </signal>
 <signal name="MOSFET_DAC">
