File: hardware/recorder/Recorder.brd (EAGLE design)
At the start: 72.6 x 77.2 mm, 42 parts, among them T1 VN0109N3-G-ND, T2 IRF1404PBF, U1 DEV-16771_REDUCED_PINS, U2 MCP4822-E/P, U3 LM6132BIN, U4 Value, U5 L7808ABV, U6 L7908CV

Commit message: Add minor changes to the hardware
Parts:
- R_SHUNT: value 1R -> 2R
- moved C5 0.51 mm to (56.9, 13.2)
- moved C2 0.25 mm to (28.7, 20.6)
- moved C3 0.25 mm to (26.2, 20.6)
Routing:
- net +5V: track 66.1 -> 64.9 mm
- net +8V: track 63.8 -> 64.3 mm
Changed lines of the file:
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@@
 <attribute name="TYPE" value="TYPE" x="65.024" y="29.972" size="1.778" layer="27" rot="R270" display="off"/>
 </element>
-<element name="R_SHUNT" library="rcl" library_urn="urn:adsk.eagle:library:334" package="0207/10" package3d_urn="urn:adsk.eagle:package:23491/2" value="1R" x="54.356" y="27.94" smashed="yes">
+<element name="R_SHUNT" library="rcl" library_urn="urn:adsk.eagle:library:334" package="0207/10" package3d_urn="urn:adsk.eagle:package:23491/2" value="2R" x="54.356" y="27.94" smashed="yes">
 <attribute name="NAME" x="54.61" y="29.464" size="1.016" layer="25" ratio="10"/>
 <attribute name="POPULARITY" value="81" x="35.56" y="44.196" size="1.778" layer="27" display="off"/>
@@
 <attribute name="VALUE" x="30.032" y="54.136" size="1.016" layer="25"/>
 </element>
-<element name="C3" library="rcl" library_urn="urn:adsk.eagle:library:334" package="C025-024X044" package3d_urn="urn:adsk.eagle:package:23630/1" value="0.1u" x="26.162" y="20.32" smashed="yes" rot="R90">
-<attribute name="NAME" x="24.765" y="18.288" size="1.016" layer="25" ratio="10" rot="R90"/>
-<attribute name="POPULARITY" value="56" x="26.162" y="20.32" size="1.778" layer="27" rot="R90" display="off"/>
-<attribute name="SPICEPREFIX" value="C" x="26.162" y="20.32" size="1.778" layer="27" rot="R90" display="off"/>
-<attribute name="VALUE" x="23.749" y="23.368" size="1.016" layer="25" ratio="10" rot="R270"/>
-</element>
-<element name="C2" library="rcl" library_urn="urn:adsk.eagle:library:334" package="C025-024X044" package3d_urn="urn:adsk.eagle:package:23630/1" value="10u" x="28.702" y="20.32" smashed="yes" rot="R90">
-<attribute name="NAME" x="31.115" y="19.558" size="1.016" layer="25" ratio="10" rot="R90"/>
-<attribute name="POPULARITY" value="56" x="28.702" y="20.32" size="1.778" layer="27" rot="R90" display="off"/>
-<attribute name="SPICEPREFIX" value="C" x="28.702" y="20.32" size="1.778" layer="27" rot="R90" display="off"/>
-<attribute name="VALUE" x="30.099" y="23.876" size="1.016" layer="25" ratio="10" rot="R180"/>
-</element>
-<element name="C5" library="rcl" library_urn="urn:adsk.eagle:library:334" package="C025-024X044" package3d_urn="urn:adsk.eagle:package:23630/1" value="0.1u" x="56.896" y="13.716" smashed="yes">
-<attribute name="NAME" x="60.579" y="12.954" size="1.016" layer="25" ratio="10" rot="R90"/>
-<attribute name="POPULARITY" value="56" x="56.896" y="13.716" size="1.778" layer="27" display="off"/>
-<attribute name="SPICEPREFIX" value="C" x="56.896" y="13.716" size="1.778" layer="27" display="off"/>
-<attribute name="VALUE" x="55.626" y="11.049" size="1.016" layer="25" ratio="10"/>
+<element name="C3" library="rcl" library_urn="urn:adsk.eagle:library:334" package="C025-024X044" package3d_urn="urn:adsk.eagle:package:23630/1" value="0.1u" x="26.162" y="20.574" smashed="yes" rot="R90">
+<attribute name="NAME" x="24.765" y="18.542" size="1.016" layer="25" ratio="10" rot="R90"/>
+<attribute name="POPULARITY" value="56" x="26.162" y="20.574" size="1.778" layer="27" rot="R90" display="off"/>
+<attribute name="SPICEPREFIX" value="C" x="26.162" y="20.574" size="1.778" layer="27" rot="R90" display="off"/>
+<attribute name="VALUE" x="23.749" y="23.622" size="1.016" layer="25" ratio="10" rot="R270"/>
+</element>
+<element name="C2" library="rcl" library_urn="urn:adsk.eagle:library:334" package="C025-024X044" package3d_urn="urn:adsk.eagle:package:23630/1" value="10u" x="28.702" y="20.574" smashed="yes" rot="R90">
+<attribute name="NAME" x="31.115" y="19.812" size="1.016" layer="25" ratio="10" rot="R90"/>
+<attribute name="POPULARITY" value="56" x="28.702" y="20.574" size="1.778" layer="27" rot="R90" display="off"/>
+<attribute name="SPICEPREFIX" value="C" x="28.702" y="20.574" size="1.778" layer="27" rot="R90" display="off"/>
+<attribute name="VALUE" x="30.099" y="24.13" size="1.016" layer="25" ratio="10" rot="R180"/>
+</element>
+<element name="C5" library="rcl" library_urn="urn:adsk.eagle:library:334" package="C025-024X044" package3d_urn="urn:adsk.eagle:package:23630/1" value="0.1u" x="56.896" y="13.208" smashed="yes">
+<attribute name="NAME" x="60.579" y="12.446" size="1.016" layer="25" ratio="10" rot="R90"/>
+<attribute name="POPULARITY" value="56" x="56.896" y="13.208" size="1.778" layer="27" display="off"/>
+<attribute name="SPICEPREFIX" value="C" x="56.896" y="13.208" size="1.778" layer="27" display="off"/>
+<attribute name="VALUE" x="55.626" y="10.541" size="1.016" layer="25" ratio="10"/>
 </element>
 <element name="C6" library="rcl" library_urn="urn:adsk.eagle:library:334" package="C025-024X044" package3d_urn="urn:adsk.eagle:package:23630/1" value="0.1u" x="46.482" y="24.13" smashed="yes" rot="R180">
@@
 <wire x1="55.626" y1="17.653" x2="55.626" y2="16.51" width="1.27" layer="1"/>
 <wire x1="26.416" y1="39.878" x2="29.05" y2="39.878" width="1.27" layer="1"/>
-<wire x1="55.626" y1="13.716" x2="55.626" y2="16.51" width="1.27" layer="1"/>
+<wire x1="55.626" y1="13.208" x2="55.626" y2="16.51" width="1.27" layer="1"/>
 <contactref element="C8" pad="2"/>
 <wire x1="51.308" y1="35.052" x2="51.308" y2="39.624" width="1.27" layer="1"/>
@@
 <wire x1="27.305" y1="65.024" x2="27.227" y2="64.946" width="1.27" layer="1"/>
 <wire x1="27.227" y1="64.946" x2="27.227" y2="61.666" width="1.27" layer="1"/>
-<wire x1="26.162" y1="19.05" x2="26.162" y2="16.635" width="1.27" layer="1"/>
+<wire x1="26.162" y1="19.304" x2="26.162" y2="16.635" width="1.27" layer="1"/>
 <wire x1="26.162" y1="16.635" x2="26.037" y2="16.51" width="1.27" layer="1"/>
-<wire x1="28.702" y1="19.05" x2="26.162" y2="16.51" width="1.27" layer="1"/>
-<wire x1="26.162" y1="16.51" x2="26.037" y2="16.51" width="1.27" layer="1"/>
 <wire x1="27.227" y1="61.666" x2="21.844" y2="56.283" width="1.27" layer="1"/>
 <wire x1="21.844" y1="56.283" x2="21.844" y2="37.719" width="1.27" layer="1"/>
 <wire x1="21.844" y1="37.719" x2="23.622" y2="35.941" width="1.27" layer="1"/>
-<wire x1="26.162" y1="19.304" x2="26.162" y2="19.05" width="1.27" layer="1"/>
 <wire x1="26.162" y1="19.304" x2="23.622" y2="21.844" width="1.27" layer="1"/>
 <wire x1="23.622" y1="35.941" x2="23.622" y2="21.844" width="1.27" layer="1"/>
+<wire x1="26.162" y1="19.304" x2="28.702" y2="19.304" width="1.27" layer="1"/>
 </signal>
 <signal name="N$5">
