File: hardware/recorder/Recorder.sch (EAGLE design)
At the start: 23 parts, among them U1 PDM1-S5-D12-S, U2 LM6132BIN, U3 Value, U4 L7908CV, U5 L7808ABV, U6 ZVN4424A, U7 TEENSY_3.6_DIL

Commit message: Update recorder hardware
Parts:
- R3: value 300R -> 330R
- renumbered HARVESTER to HARVESTER_TERMINAL
Other:
- note added: "Author: S.Mosavat"
- note added: "I_max_record = 3.3 / (R_shunt * GAIN_ia) GAIN_ia = 1 + (50k / R_GAIN)"
- note added: "SOCRAETES Emulator"
- note added: "University of Duisburg-Essens Networked Embedded Systems Group (NES) https://www.nes.uni-due.de/"
- note added: "V 1.1.4"
Changed lines of the file:
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@@
 <parts>
 <part name="U1" library="PDM1-S5-D12-S" deviceset="PDM1-S5-D12-S" device=""/>
-<part name="HARVESTER" library="con-ptr500" library_urn="urn:adsk.eagle:library:181" deviceset="AK300/2" device="" package3d_urn="urn:adsk.eagle:package:9881/1"/>
+<part name="HARVESTER_TERMINAL" library="con-ptr500" library_urn="urn:adsk.eagle:library:181" deviceset="AK300/2" device="" package3d_urn="urn:adsk.eagle:package:9881/1"/>
 <part name="D1" library="diode" library_urn="urn:adsk.eagle:library:210" deviceset="ZENER-DIODE" device="ZD-7.5" package3d_urn="urn:adsk.eagle:package:43411/1" value="3v3"/>
 <part name="U2" library="LM6132BIN" deviceset="LM6132BIN" device=""/>
@@
 <part name="+3V2" library="supply1" library_urn="urn:adsk.eagle:library:371" deviceset="+3V3" device=""/>
 <part name="SUPPLY21" library="supply2" library_urn="urn:adsk.eagle:library:372" deviceset="GND" device=""/>
-<part name="R3" library="rcl" library_urn="urn:adsk.eagle:library:334" deviceset="R-EU_" device="0207/10" package3d_urn="urn:adsk.eagle:package:23491/2" value="300R"/>
+<part name="R3" library="rcl" library_urn="urn:adsk.eagle:library:334" deviceset="R-EU_" device="0207/10" package3d_urn="urn:adsk.eagle:package:23491/2" value="330R"/>
 <part name="LED_PWR" library="led" library_urn="urn:adsk.eagle:library:259" deviceset="LED" device="5MM" package3d_urn="urn:adsk.eagle:package:15799/2"/>
 <part name="R4" library="rcl" library_urn="urn:adsk.eagle:library:334" deviceset="R-EU_" device="0207/10" package3d_urn="urn:adsk.eagle:package:23491/2" value="1k"/>
@@
 <sheet>
 <plain>
+<text x="215.9" y="20.32" size="2.54" layer="94">SOCRAETES Emulator</text>
+<text x="215.9" y="15.24" size="2.54" layer="94">V 1.1.4</text>
+<text x="215.9" y="10.16" size="2.54" layer="94">Author: S.Mosavat</text>
+<text x="162.56" y="7.62" size="2.54" layer="94">University of Duisburg-Essens
+Networked Embedded Systems
+Group (NES)
+https://www.nes.uni-due.de/</text>
+<text x="43.18" y="104.14" size="1.778" layer="97">I_max_record = 3.3 / (R_shunt * GAIN_ia)
+GAIN_ia = 1 + (50k / R_GAIN)</text>
 </plain>
 <instances>
@@
 <attribute name="VALUE" x="175.2477" y="149.8477" size="2.54308125" layer="96" align="top-left"/>
 </instance>
-<instance part="HARVESTER" gate="-1" x="132.08" y="20.32" smashed="yes" rot="R270">
+<instance part="HARVESTER_TERMINAL" gate="-1" x="132.08" y="20.32" smashed="yes" rot="R270">
 <attribute name="NAME" x="132.969" y="21.59" size="1.778" layer="95" rot="R90"/>
 </instance>
-<instance part="HARVESTER" gate="-2" x="127" y="20.32" smashed="yes" rot="R270">
+<instance part="HARVESTER_TERMINAL" gate="-2" x="127" y="20.32" smashed="yes" rot="R270">
 <attribute name="NAME" x="127.889" y="21.59" size="1.778" layer="95" rot="R90"/>
 <attribute name="VALUE" x="123.317" y="24.13" size="1.778" layer="96" rot="R270"/>
@@
 <attribute name="VALUE" x="46.99" y="120.142" size="1.778" layer="96" rot="R180"/>
 </instance>
-<instance part="FRAME1" gate="G$1" x="0" y="0" smashed="yes">
-<attribute name="DRAWING_NAME" x="217.17" y="15.24" size="2.54" layer="94"/>
-<attribute name="LAST_DATE_TIME" x="217.17" y="10.16" size="2.286" layer="94"/>
-<attribute name="SHEET" x="230.505" y="5.08" size="2.54" layer="94"/>
-</instance>
+<instance part="FRAME1" gate="G$1" x="0" y="0" smashed="yes"/>
 <instance part="U5" gate="A" x="241.3" y="109.22" smashed="yes" rot="R180">
 <attribute name="NAME" x="220.6244" y="107.7214" size="2.0828" layer="95" ratio="6" rot="SR180"/>
@@
 </segment>
 <segment>
-<pinref part="HARVESTER" gate="-2" pin="KL"/>
+<pinref part="HARVESTER_TERMINAL" gate="-2" pin="KL"/>
 <pinref part="SUPPLY15" gate="GND" pin="GND"/>
 </segment>
@@
 <pinref part="U1" gate="G$1" pin="-VO"/>
 <pinref part="C3" gate="G$1" pin="-"/>
-<wire x1="203.2" y1="160.02" x2="213.36" y2="160.02" width="0.1524" layer="91"/>
+<wire x1="203.2" y1="160.02" x2="214.675275" y2="160.02" width="0.1524" layer="91"/>
 <pinref part="P-1" gate="1" pin="-12V"/>
 <wire x1="214.675275" y1="160.02" x2="220.98" y2="160.02" width="0.1524" layer="91"/>
 <wire x1="214.675275" y1="158.317796875" x2="214.675275" y2="160.02" width="0.1524" layer="91"/>
-<wire x1="214.675275" y1="160.02" x2="213.36" y2="160.02" width="0.1524" layer="91"/>
 </segment>
 <segment>
@@
 <net name="HARVESTER+" class="0">
 <segment>
-<pinref part="HARVESTER" gate="-1" pin="KL"/>
+<pinref part="HARVESTER_TERMINAL" gate="-1" pin="KL"/>
 <wire x1="132.08" y1="15.24" x2="132.08" y2="12.7" width="0.1524" layer="91"/>
 <label x="129.54" y="10.16" size="1.778" layer="95"/>
@@
 </drawing>
 <compatibility>
+<note version="6.3" minversion="6.2.2" severity="warning">
+Since Version 6.2.2 text objects can contain more than one line,
+which will not be processed correctly with this version.
+</note>
 <note version="8.2" severity="warning">
 Since Version 8.2, EAGLE supports online libraries. The ids

Commit message: Add minor changes to the schematics
Other:
- note added: "University of Duisburg-Essen Networked Embedded Systems Group (NES) https://www.nes.uni-due.de/"
- note removed: "University of Duisburg-Essens Networked Embedded Systems Group (NES) https://www.nes.uni-due.de/"
Changed lines of the file:
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@@
 <text x="215.9" y="15.24" size="2.54" layer="94">V 1.1.4</text>
 <text x="215.9" y="10.16" size="2.54" layer="94">Author: S.Mosavat</text>
-<text x="162.56" y="7.62" size="2.54" layer="94">University of Duisburg-Essens
+<text x="162.56" y="7.62" size="2.54" layer="94">University of Duisburg-Essen
 Networked Embedded Systems
 Group (NES)

Commit message: Migrate recorder board to Teensy 4.1
Parts:
- removed D1, D2: 3v3, diode:ZENER-DIODEZD-7.5
- removed LED_PWR: (no value), led:LED5MM
- removed R_GAIN: (no value), rcl:R-EU_0207/10
- added C10: EDS224Z3R6H, SamacSys_Parts:EDS224Z3R6H
- added C11: 0.33u, rcl:C-EU025-024X044
- added C12, C7, C9: 0.1u, rcl:C-EU025-024X044
- added C13: 2.2u, rcl:C-EU025-024X044
- added C14: 1u, rcl:C-EU025-024X044
- added C8: 10u, rcl:C-EU025-024X044
- added D3: 1N5817-B, diode:1N5817-B
- added GAIN_SELECT: (no value), con-lstb:MA04-2
- added MODE: (no value), con-lstb:MA03-1
- added POWER, STATUS: (no value), led:LED5MM
- added PS1: RD-0512D, RD-0512D:RD-0512D
- added R5: 330R, rcl:R-EU_0207/10
- added R_GAIN_100: 511R, rcl:R-EU_0207/10
- added R_GAIN_200: 249R, rcl:R-EU_0207/10
- added R_GAIN_25: 2k1, rcl:R-EU_0207/10
- added R_GAIN_50: 1k02, rcl:R-EU_0207/10
- added U8: DEV-16771_REDUCED_PINS, DEV-16771 (Teensy 41):DEV-16771_REDUCED_PINS
- C1, C5, C6: device rcl:CPOL-EUE2-4 -> rcl:C-EU025-024X044
- C2, C3: device rcl:CPOL-EUE2-5 -> rcl:C-EU025-024X044
- C4: value 1u -> 0.1u; device rcl:CPOL-EUE2-5 -> rcl:C-EU025-024X044
- R_SHUNT: value (none) -> 1R
- U1: value PDM1-S5-D12-S -> MCP4822-E/P; device PDM1-S5-D12-S:PDM1-S5-D12-S -> MCP4822-E_P:MCP4822-E/P
- U7: value TEENSY_3.6_DIL -> ZVN4424A; device Teensy_3_and_LC_Series_Boards_v1.4:TEENSY_3.6_DIL -> NES_Solar_Cell_Recorder_And_Emulator:ZVN4424A
Connections:
- removed net MOSFET_DAC: R4.2, U7.A21/DAC0
- removed net N$4: D1.C, D2.A
- new net +5V: C1.1, C7.1, C8.1, PS1.+VIN, U1.VDD, U8.VIN
- new net CURRENT_SENSE_AMP_OUTPUT: U3.OUT, U8.A14
- new net DAC_CS: U1.!CS, U8.RX8
- new net DAC_MOSI: U1.SDI, U8.MOSI
- new net DAC_SCK: U1.SCK, U8.SCK
- new net HARVESTER_VOLTAGE_DIVIDER_OUTPUT: R1.1, R2.2, U8.A15
- new net JUMPER_SELECT_MODE: MODE.2, U8.OUT1B
- new net MOSFET_DAC_OUTPUT: R4.2, U1.VOUTA
- new net N$12: R_GAIN_100.2, R_GAIN_200.2, R_GAIN_25.2, R_GAIN_50.2, U3.RG_2
- new net N$13: GAIN_SELECT.1, GAIN_SELECT.3, GAIN_SELECT.5, GAIN_SELECT.7, U3.RG
- new net N$14: GAIN_SELECT.2, R_GAIN_200.1
- new net STATUS_LED: R5.2, U8.TX1
- net +12V: now also C11.1, C2.1, PS1.+VOUT; no longer C2.+, U1.+VO
- net +3V3: now also D3.A, MODE.3, U8.3.3V; no longer U7.3.3V
- net +8V: now also C12.2, C5.1, C9.1; no longer C5.+
- net -12V: now also C13.2, C3.1, PS1.-VOUT; no longer C3.-, U1.-VO
- net -8V: now also C14.2, C4.1; no longer C4.-
- net GND: now also C1.2, C10.-, C11.2, C12.1, C13.1, C14.1, C2.2, C3.2, C4.2, C5.2, C6.2, C7.2, C8.2, C9.2, MODE.1, POWER.C, PS1.-VIN, PS1.COM, STATUS.C, U1.!LDAC, U1.AVSS, U7.S, U8.GND; no longer C1.-, C2.-, C3.+, C4.+, C5.-, C6.-, D1.A, LED_PWR.C, U1.0V, U1.GND, U7.GND
- net HARVESTER+: now also C6.1; no longer C6.+, D2.C
- net N$1: now also GAIN_SELECT.8, R_GAIN_25.1; no longer R_GAIN.2, U3.RG_2
- net N$10: now also GAIN_SELECT.4, R_GAIN_100.1; no longer U3.OUT, U7.17/A3/T/PWM
- net N$11: now also U7.G
- net N$2: now also C10.+, D3.C, U8.VBAT; no longer C1.+, U1.VIN, U7.VIN
- net N$3: now also GAIN_SELECT.6, R_GAIN_50.1; no longer R_GAIN.1, U3.RG
- net N$6: now also U7.D
- net N$7: now also R5.1, STATUS.A; no longer R1.1, R2.2, U7.16/A2/T/PWM
- net N$9: now also POWER.A; no longer LED_PWR.A
Other:
- note added: "I_max_record = 3.3 / (R_shunt * GAIN_ia) GAIN_ia = 1 + (50k / R_GAIN) With R_shunt = 2R: GAIN_ia = 25: I_max_record = 66 mA GAIN_ia = 50: I_max_record = 33 mA GAIN_ia = 100: I_max_record = 16.5 mA GAIN_ia = 200: I_max_record = 8.25 mA"
- note added: "SOCRAETES Recorder"
- note added: "v0.2.6"
- note removed: "I_max_record = 3.3 / (R_shunt * GAIN_ia) GAIN_ia = 1 + (50k / R_GAIN)"
- note removed: "SOCRAETES Emulator"
- note removed: "V 1.1.4"

Commit message: Add error LED to the board
Parts:
- added ERROR: (no value), led:LED5MM
- added R6: 330R, rcl:R-EU_0207/10
Connections:
- new net ERROR_LED: R6.2, U8.OUT2
- new net N$4: ERROR.A, R6.1
- net GND: now also ERROR.C
Changed lines of the file:
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@@
 <part name="C12" library="rcl" library_urn="urn:adsk.eagle:library:334" deviceset="C-EU" device="025-024X044" package3d_urn="urn:adsk.eagle:package:23630/1" value="0.1u"/>
 <part name="SUPPLY30" library="supply2" library_urn="urn:adsk.eagle:library:372" deviceset="GND" device=""/>
+<part name="SUPPLY31" library="supply2" library_urn="urn:adsk.eagle:library:372" deviceset="GND" device=""/>
+<part name="R6" library="rcl" library_urn="urn:adsk.eagle:library:334" deviceset="R-EU_" device="0207/10" package3d_urn="urn:adsk.eagle:package:23491/2" value="330R"/>
+<part name="ERROR" library="led" library_urn="urn:adsk.eagle:library:259" deviceset="LED" device="5MM" package3d_urn="urn:adsk.eagle:package:15799/2"/>
 </parts>
 <sheets>
@@
 </segment>
 </net>
+<net name="ERROR_LED" class="0">
+<segment>
+<pinref part="U8" gate="G$1" pin="OUT2"/>
+<wire x1="132.08" y1="114.3" x2="134.62" y2="114.3" width="0.1524" layer="91"/>
+<label x="134.62" y="114.3" size="1.778" layer="95" xref="yes"/>
+</segment>
+</net>
 </nets>
 </sheet>
@@
 <attribute name="VALUE" x="69.215" y="126.365" size="1.778" layer="96"/>
 </instance>
+<instance part="SUPPLY31" gate="GND" x="109.22" y="17.78" smashed="yes">
+<attribute name="VALUE" x="112.395" y="17.145" size="1.778" layer="96"/>
+</instance>
+<instance part="R6" gate="G$1" x="109.22" y="38.1" smashed="yes" rot="R90">
+<attribute name="NAME" x="107.7214" y="34.29" size="1.778" layer="95" rot="R90"/>
+<attribute name="VALUE" x="112.522" y="34.29" size="1.778" layer="96" rot="R90"/>
+</instance>
+<instance part="ERROR" gate="G$1" x="109.22" y="27.94" smashed="yes">
+<attribute name="NAME" x="105.156" y="20.828" size="1.778" layer="95" rot="R90"/>
+<attribute name="VALUE" x="114.935" y="23.368" size="1.778" layer="96" rot="R90"/>
+</instance>
 </instances>
 <busses>
@@
 <wire x1="71.12" y1="134.62" x2="76.2" y2="134.62" width="0.1524" layer="91"/>
 </segment>
+<segment>
+<pinref part="SUPPLY31" gate="GND" pin="GND"/>
+<pinref part="ERROR" gate="G$1" pin="C"/>
+<wire x1="109.22" y1="20.32" x2="109.22" y2="22.86" width="0.1524" layer="91"/>
+</segment>
 </net>
 <net name="HARVESTER+" class="0">
@@
 </segment>
 </net>
+<net name="N$4" class="0">
+<segment>
+<pinref part="R6" gate="G$1" pin="1"/>
+<pinref part="ERROR" gate="G$1" pin="A"/>
+<wire x1="109.22" y1="33.02" x2="109.22" y2="30.48" width="0.1524" layer="91"/>
+</segment>
+</net>
+<net name="ERROR_LED" class="0">
+<segment>
+<pinref part="R6" gate="G$1" pin="2"/>
+<wire x1="109.22" y1="43.18" x2="109.22" y2="45.72" width="0.1524" layer="91"/>
+<label x="109.22" y="45.72" size="1.778" layer="95" rot="R90" xref="yes"/>
+</segment>
+</net>

Commit message: Add minor changes to the hardware
Changed lines of the file:
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@@
 <instance part="U2" gate="A" x="66.04" y="45.72" smashed="yes">
 <attribute name="NAME" x="63.5" y="59.42" size="2.0828" layer="95" ratio="10" rot="SR0"/>
-<attribute name="VALUE" x="53.34" y="29.02" size="2.0828" layer="96" ratio="10" rot="SR0"/>
+<attribute name="VALUE" x="60.96" y="29.02" size="2.0828" layer="96" ratio="10" rot="SR0"/>
 </instance>
 <instance part="SUPPLY13" gate="+8V" x="101.6" y="66.04" smashed="yes">
@@
 <instance part="U1" gate="A" x="73.66" y="129.54" smashed="yes">
 <attribute name="NAME" x="60.96" y="143.24" size="2.0828" layer="95" ratio="10" rot="SR0"/>
-<attribute name="VALUE" x="63.5" y="112.84" size="2.0828" layer="96" ratio="10" rot="SR0"/>
+<attribute name="VALUE" x="66.04" y="112.84" size="2.0828" layer="96" ratio="10" rot="SR0"/>
 </instance>
 <instance part="SUPPLY24" gate="GND" x="93.98" y="111.76" smashed="yes">

Commit message: Update part designators
Parts:
- removed U8: DEV-16771_REDUCED_PINS, DEV-16771 (Teensy 41):DEV-16771_REDUCED_PINS
- added T1: ZVN4424A, NES_Solar_Cell_Recorder_And_Emulator:ZVN4424A
- C1: value 2.2u -> EDS224Z3R6H; device rcl:C-EU025-024X044 -> SamacSys_Parts:EDS224Z3R6H
- C10: value EDS224Z3R6H -> 0.33u; device SamacSys_Parts:EDS224Z3R6H -> rcl:C-EU025-024X044
- C11: value 0.33u -> 1u
- C12, C9: value 0.1u -> 2.2u
- C13: value 2.2u -> 1u
- C2: value 1u -> 10u
- C3: value 1u -> 0.1u
- C8: value 10u -> 0.1u
- R3: value 330R -> 1k
- R4: value 1k -> 330R
- U1: value MCP4822-E/P -> DEV-16771_REDUCED_PINS; device MCP4822-E_P:MCP4822-E/P -> DEV-16771 (Teensy 41):DEV-16771_REDUCED_PINS
- U2: value LM6132BIN -> MCP4822-E/P; device LM6132BIN:LM6132BIN -> MCP4822-E_P:MCP4822-E/P
- U3: value Value -> LM6132BIN; device INA121PA:INA121PA -> LM6132BIN:LM6132BIN
- U4: value L7908CV -> Value; device L7908CV:L7908CV -> INA121PA:INA121PA
- U6: value ZVN4424A -> L7908CV; device NES_Solar_Cell_Recorder_And_Emulator:ZVN4424A -> L7908CV:L7908CV
- renumbered D3 to D1, U7 to T2
Connections:
- net +12V: now also C10.1, C13.1; no longer C11.1, C2.1
- net +3V3: now also R4.2, U1.3.3V; no longer R3.2, U8.3.3V
- net +5V: now also C12.1, C2.1, C3.1, U1.VIN, U2.VDD; no longer C1.1, C7.1, C8.1, U1.VDD, U8.VIN
- net +8V: now also C4.1, C8.2, U3.+V, U4.V+; no longer C12.2, C9.1, U2.+V, U3.V+
- net -12V: now also C14.1, C9.2, U6.IN; no longer C13.2, C3.1, U4.IN
- net -8V: now also C11.2, C6.1, U4.V-, U6.OUT; no longer C14.2, C4.1, U3.V-, U4.OUT
- net CURRENT_SENSE_AMP_OUTPUT: now also U1.A14, U4.OUT; no longer U3.OUT, U8.A14
- net DAC_CS: now also U1.RX8, U2.!CS; no longer U1.!CS, U8.RX8
- net DAC_MOSI: now also U1.MOSI, U2.SDI; no longer U1.SDI, U8.MOSI
- net DAC_SCK: now also U2.SCK; no longer U8.SCK
- net ERROR_LED: now also U1.OUT2; no longer U8.OUT2
- net GND: now also C1.-, C10.2, C11.1, C12.2, C13.2, C14.2, C8.1, C9.1, T1.S, U1.GND, U2.!LDAC, U2.AVSS, U3.+INB, U3.-V, U4.REF, U6.GND; no longer C1.2, C10.-, C11.2, C12.1, C13.1, C14.1, C8.2, C9.2, U1.!LDAC, U1.AVSS, U2.+INB, U2.-V, U3.REF, U4.GND, U6.S, U8.GND
- net HARVESTER+: now also C7.1, U3.+INA, U4.IN+; no longer C6.1, U2.+INA, U3.IN+
- net HARVESTER_VOLTAGE_DIVIDER_OUTPUT: now also U1.A15; no longer U8.A15
- net JUMPER_SELECT_MODE: now also U1.OUT1B; no longer U8.OUT1B
- net MOSFET_DAC_OUTPUT: now also R3.2, U2.VOUTA; no longer R4.2, U1.VOUTA
- net N$11: now also R3.1, T1.G; no longer R4.1, U6.G
- net N$12: now also U4.RG_2; no longer U3.RG_2
- net N$13: now also U4.RG; no longer U3.RG
- net N$2: now also C1.+, U1.VBAT; no longer C10.+, U8.VBAT
- net N$5: now also U3.-INB, U3.OUT_B; no longer U2.-INB, U2.OUT_B
- net N$6: now also T1.D, U4.IN-; no longer U3.IN-, U6.D
- net N$8: now also U3.-INA, U3.OUT_A; no longer U2.-INA, U2.OUT_A
- net N$9: now also R4.1; no longer R3.1
- net STATUS_LED: now also U1.TX1; no longer U8.TX1
